File: pcb/_autosave-Numpad.kicad_pcb (KiCad board)
At the start: 2 copper layers, 61 parts, among them P1 USB-MICRO-B, SW1 F13, SW10 8, SW11 9, SW12 PLUS, SW13 4, SW14 5, SW15 6, SW16 ENTER, SW17 1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

Commit message: Try routing one row, one column
Parts:
- removed P2, P3, P4, P5: , Connect:1pin
- SW1: value F13 -> F1
- SW2: value F14 -> F2
- SW3: value F16 -> F3
- SW4: value F15 -> F4
- moved D13 4.21 mm to (71.2, 132.8), turned to 90 degrees
- moved D5 4.21 mm to (71.2, 94.7), turned to 90 degrees
- moved D1 4.09 mm to (71.2, 75.4), turned to 90 degrees
- moved D17 4.09 mm to (71.2, 151.6), turned to 90 degrees
- moved D9 4.09 mm to (71.2, 113.5), turned to 90 degrees
Routing:
- net Net-(D5-Pad2): track 0.00 -> 10.6 mm
- net Net-(D1-Pad2): track 0.00 -> 10.4 mm
