File: pcb/Numpad.sch (KiCad schematic (older format))
At the start: 57 parts, among them P1 USB-MICRO-B, P2 Header, SW1 F1, SW10 8, SW11 9, SW12 PLUS, SW13 4, SW14 5, SW15 6, SW16 ENTER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

Commit message: Update schematic
Parts:
- removed P2: Header, Socket_Strips:Socket_Strip_Angled_2x03, symbol CONN_02X03
- added SW22: SW_PUSH, symbol SW_PUSH
- C2, C3: value 22p -> 18p
- C4, C5: value 100n -> 0.1u
- C6: value 4u7 -> 1u
- R3: value 100 -> 1K
- Y1: value CRYSTAL -> 16MHz
Connections:
- net labels added: VCC
- net labels removed: ISP_MISO, ISP_MOSI, ISP_SCK
- wire segments 73 -> 69
Changed lines of the file:
@@
 LIBS:contrib
 LIBS:valves
-LIBS:Numpad-cache
 EELAYER 25 0
 EELAYER END
@@
 Text Label 8300 1000 0    60   ~ 0
 ROW0
+Text Label 8300 1100 0    60   ~ 0
+ROW1
+Text Label 8300 1200 0    60   ~ 0
+ROW2
+Text Label 8300 1300 0    60   ~ 0
+ROW3
 Text Label 8300 1400 0    60   ~ 0
-ROW1
-Text Label 8300 1500 0    60   ~ 0
-ROW2
-Text Label 8300 1600 0    60   ~ 0
-ROW3
-Text Label 8300 1700 0    60   ~ 0
 ROW4
 Text Label 8300 2200 0    60   ~ 0
@@
 P 7700 6150
 F 0 "R3" V 7621 6150 50  0000 C CNN
-F 1 "100" V 7700 6150 50  0000 C CNN
+F 1 "1K" V 7700 6150 50  0000 C CNN
 F 2 "Keyboard:R_0805" V 7630 6150 50  0001 C CNN
 F 3 "" H 7700 6150 50  0000 C CNN
@@
 P 5650 5150
 F 0 "C2" H 5675 5250 50  0000 L CNN
-F 1 "22p" H 5675 5050 50  0000 L CNN
+F 1 "18p" H 5675 5050 50  0000 L CNN
 F 2 "Keyboard:C_0805" H 5688 5000 50  0001 C CNN
 F 3 "" H 5650 5150 50  0000 C CNN
@@
 P 6450 5150
 F 0 "C3" H 6475 5250 50  0000 L CNN
-F 1 "22p" H 6475 5050 50  0000 L CNN
+F 1 "18p" H 6475 5050 50  0000 L CNN
 F 2 "Keyboard:C_0805" H 6488 5000 50  0001 C CNN
 F 3 "" H 6450 5150 50  0000 C CNN
@@
 P 6050 4850
 F 0 "Y1" H 6050 5000 50  0000 C CNN
-F 1 "CRYSTAL" H 6050 4700 50  0000 C CNN
+F 1 "16MHz" H 6050 4700 50  0000 C CNN
 F 2 "Crystals:Crystal_HC49-U_Vertical" H 6050 4850 50  0001 C CNN
 F 3 "" H 6050 4850 50  0000 C CNN
@@
 L +5V #PWR08
 U 1 1 57D6C60C
-P 5700 800
-F 0 "#PWR08" H 5700 650 50  0001 C CNN
-F 1 "+5V" H 5700 940 50  0000 C CNN
-F 2 "" H 5700 800 50  0000 C CNN
-F 3 "" H 5700 800 50  0000 C CNN
-	1    5700 800
-	1    0    0    -1
-$EndComp
-$Comp
-L CONN_02X03 P2
-U 1 1 57D6CEBD
-P 8250 5200
-F 0 "P2" H 8250 5400 50  0000 C CNN
-F 1 "Header" H 8250 5000 50  0001 C CNN
-F 2 "Socket_Strips:Socket_Strip_Angled_2x03" H 8250 4000 50  0001 C CNN
-F 3 "" H 8250 4000 50  0000 C CNN
-	1    8250 5200
+P 5850 1000
+F 0 "#PWR08" H 5850 850 50  0001 C CNN
+F 1 "+5V" H 5850 1140 50  0000 C CNN
+F 2 "" H 5850 1000 50  0000 C CNN
+F 3 "" H 5850 1000 50  0000 C CNN
+	1    5850 1000
 	1    0    0    -1
 $EndComp
@@
 $EndComp
 $Comp
-L +5V #PWR09
-U 1 1 57D6D2B3
-P 6050 2700
-F 0 "#PWR09" H 6050 2550 50  0001 C CNN
-F 1 "+5V" H 6050 2840 50  0000 C CNN
-F 2 "" H 6050 2700 50  0000 C CNN
-F 3 "" H 6050 2700 50  0000 C CNN
-	1    6050 2700
-	1    0    0    -1
-$EndComp
-Text Label 8300 1100 0    60   ~ 0
-ISP_SCK
-Text Label 8300 1200 0    60   ~ 0
-ISP_MOSI
-Text Label 8300 1300 0    60   ~ 0
-ISP_MISO
-Text Label 8000 5200 2    60   ~ 0
-ISP_SCK
-Text Label 8750 5200 0    60   ~ 0
-ISP_MOSI
-Text Label 8000 5100 2    60   ~ 0
-ISP_MISO
-$Comp
-L GND #PWR010
-U 1 1 57D706F1
-P 8650 5300
-F 0 "#PWR010" H 8650 5050 50  0001 C CNN
-F 1 "GND" H 8650 5150 50  0000 C CNN
-F 2 "" H 8650 5300 50  0000 C CNN
-F 3 "" H 8650 5300 50  0000 C CNN
-	1    8650 5300
-	1    0    0    -1
-$EndComp
-$Comp
-L +5V #PWR011
-U 1 1 57D7072F
-P 8650 5100
-F 0 "#PWR011" H 8650 4950 50  0001 C CNN
-F 1 "+5V" H 8650 5240 50  0000 C CNN
-F 2 "" H 8650 5100 50  0000 C CNN
-F 3 "" H 8650 5100 50  0000 C CNN
-	1    8650 5100
-	1    0    0    -1
-$EndComp
-Text Label 8000 5300 2    60   ~ 0
-ISP_RESET
-$Comp
 L C C4
 U 1 1 57D74C20
 P 9600 5300
 F 0 "C4" H 9625 5400 50  0000 L CNN
-F 1 "100n" H 9625 5200 50  0000 L CNN
+F 1 "0.1u" H 9625 5200 50  0000 L CNN
 F 2 "Keyboard:C_0805" H 9638 5150 50  0001 C CNN
 F 3 "" H 9600 5300 50  0000 C CNN
@@
 P 10000 5300
 F 0 "C5" H 10025 5400 50  0000 L CNN
-F 1 "100n" H 10025 5200 50  0000 L CNN
+F 1 "0.1u" H 10025 5200 50  0000 L CNN
 F 2 "Keyboard:C_0805" H 10038 5150 50  0001 C CNN
 F 3 "" H 10000 5300 50  0000 C CNN
@@
 P 10400 5300
 F 0 "C6" H 10425 5400 50  0000 L CNN
-F 1 "4u7" H 10425 5200 50  0000 L CNN
+F 1 "1u" H 10425 5200 50  0000 L CNN
 F 2 "Keyboard:C_0805" H 10438 5150 50  0001 C CNN
 F 3 "" H 10400 5300 50  0000 C CNN
@@
 Connection ~ 5700 3900
 Wire Wire Line
-	5700 800  5700 1500
-Wire Wire Line
 	5700 1500 5850 1500
 Wire Wire Line
@@
 Connection ~ 5700 1100
 Wire Wire Line
-	5850 1000 5700 1000
-Connection ~ 5700 1000
-Wire Wire Line
 	6050 2700 5850 2700
-Wire Wire Line
-	8650 5100 8500 5100
-Wire Wire Line
-	8500 5200 8750 5200
-Wire Wire Line
-	8650 5300 8500 5300
 Wire Wire Line
 	5350 2000 5350 2600
@@
 	9600 5600 9600 5450
 Connection ~ 10000 5600
+$Comp
+L VCC #PWR?
+U 1 1 583F89D3
+P 9800 5000
+F 0 "#PWR?" H 9800 4850 50  0001 C CNN
+F 1 "VCC" H 9800 5150 50  0000 C CNN
+F 2 "" H 9800 5000 50  0000 C CNN
+F 3 "" H 9800 5000 50  0000 C CNN
+	1    9800 5000
+	1    0    0    -1
+$EndComp
+$Comp
+L +5V #PWR?
+U 1 1 583FB50A
+P 5850 1700
+F 0 "#PWR?" H 5850 1550 50  0001 C CNN
+F 1 "+5V" H 5850 1840 50  0000 C CNN
+F 2 "" H 5850 1700 50  0000 C CNN
+F 3 "" H 5850 1700 50  0000 C CNN
+	1    5850 1700
+	1    0    0    -1
+$EndComp
+Wire Wire Line
+	5700 1500 5700 1000
+$Comp
+L VCC #PWR?
+U 1 1 583FB754
+P 5700 1000
+F 0 "#PWR?" H 5700 850 50  0001 C CNN
+F 1 "VCC" H 5700 1150 50  0000 C CNN
+F 2 "" H 5700 1000 50  0000 C CNN
+F 3 "" H 5700 1000 50  0000 C CNN
+	1    5700 1000
+	1    0    0    -1
+$EndComp
+$Comp
+L VCC #PWR?
+U 1 1 583FE193
+P 6050 2700
+F 0 "#PWR?" H 6050 2550 50  0001 C CNN
+F 1 "VCC" H 6050 2850 50  0000 C CNN
+F 2 "" H 6050 2700 50  0000 C CNN
+F 3 "" H 6050 2700 50  0000 C CNN
+	1    6050 2700
+	1    0    0    -1
+$EndComp
+Text Label 7550 4850 2    60   ~ 0
+ISP_RESET
+$Comp
+L SW_PUSH SW22
+U 1 1 583FE502
+P 7850 4850
+F 0 "SW22" H 8000 4960 50  0000 C CNN
+F 1 "SW_PUSH" H 7850 4770 50  0000 C CNN
+F 2 "" H 7850 4850 50  0000 C CNN
+F 3 "" H 7850 4850 50  0000 C CNN
+	1    7850 4850
+	1    0    0    -1
+$EndComp
+$Comp
+L GND #PWR?
+U 1 1 583FE5A3
+P 8150 4850
+F 0 "#PWR?" H 8150 4600 50  0001 C CNN
+F 1 "GND" H 8150 4700 50  0000 C CNN
+F 2 "" H 8150 4850 50  0000 C CNN
+F 3 "" H 8150 4850 50  0000 C CNN
+	1    8150 4850
+	1    0    0    -1
+$EndComp
 $EndSCHEMATC

Commit message: Start laying out the PCB
Parts:
- removed Y1: 16MHz, Crystals:Crystal_HC49-U_Vertical, symbol Crystal
- added X1: 16MHz, Crystals:Crystal_SMD_5032_4Pads, symbol CRYSTAL_SMD
- D1, D10, D11, D12, D13, D14, D15, D16, D17, D18, D19, D2, D20, D21, D3, D4, D5, D6, D7, D8, D9: footprint Keyboard:DIODE -> Diodes_SMD:SOD-123
- D22: footprint Keyboard:LED_3MM -> Keyboard:CHERRY_MX_LED
- SW12, SW16: footprint Keyboard:CHERRY_PLATE_100H -> Keyboard:CHERRY_PLATE_200V
- SW20: footprint Keyboard:CHERRY_PLATE_100H -> Keyboard:CHERRY_PLATE_200H
- SW22: footprint (none) -> Buttons_Switches_SMD:SW_SPST_B3S-1000
Other:
- moved on the sheet: C3
Changed lines of the file:
@@
 LIBS:contrib
 LIBS:valves
+LIBS:Numpad-cache
 EELAYER 25 0
 EELAYER END
@@
 F 0 "D1" H 1300 1450 50  0000 C CNN
 F 1 "D" H 1300 1250 50  0001 C CNN
-F 2 "Keyboard:DIODE" H 1300 1350 50  0001 C CNN
+F 2 "Diodes_SMD:SOD-123" H 1300 1350 50  0001 C CNN
 F 3 "" H 1300 1350 50  0000 C CNN
 	1    1300 1350
@@
 F 0 "D2" H 2000 1450 50  0000 C CNN
 F 1 "D" H 2000 1250 50  0001 C CNN
-F 2 "Keyboard:DIODE" H 2000 1350 50  0001 C CNN
+F 2 "Diodes_SMD:SOD-123" H 2000 1350 50  0001 C CNN
 F 3 "" H 2000 1350 50  0000 C CNN
 	1    2000 1350
@@
 F 0 "D3" H 2700 1450 50  0000 C CNN
 F 1 "D" H 2700 1250 50  0001 C CNN
-F 2 "Keyboard:DIODE" H 2700 1350 50  0001 C CNN
+F 2 "Diodes_SMD:SOD-123" H 2700 1350 50  0001 C CNN
 F 3 "" H 2700 1350 50  0000 C CNN
 	1    2700 1350
@@
 F 0 "D4" H 3400 1450 50  0000 C CNN
 F 1 "D" H 3400 1250 50  0001 C CNN
-F 2 "Keyboard:DIODE" H 3400 1350 50  0001 C CNN
+F 2 "Diodes_SMD:SOD-123" H 3400 1350 50  0001 C CNN
 F 3 "" H 3400 1350 50  0000 C CNN
 	1    3400 1350
@@
 F 0 "D5" H 1300 2650 50  0000 C CNN
 F 1 "D" H 1300 2450 50  0001 C CNN
-F 2 "Keyboard:DIODE" H 1300 2550 50  0001 C CNN
+F 2 "Diodes_SMD:SOD-123" H 1300 2550 50  0001 C CNN
 F 3 "" H 1300 2550 50  0000 C CNN
 	1    1300 2550
@@
 F 0 "D6" H 2000 2650 50  0000 C CNN
 F 1 "D" H 2000 2450 50  0001 C CNN
-F 2 "Keyboard:DIODE" H 2000 2550 50  0001 C CNN
+F 2 "Diodes_SMD:SOD-123" H 2000 2550 50  0001 C CNN
 F 3 "" H 2000 2550 50  0000 C CNN
 	1    2000 2550
@@
 F 0 "D7" H 2700 2650 50  0000 C CNN
 F 1 "D" H 2700 2450 50  0001 C CNN
-F 2 "Keyboard:DIODE" H 2700 2550 50  0001 C CNN
+F 2 "Diodes_SMD:SOD-123" H 2700 2550 50  0001 C CNN
 F 3 "" H 2700 2550 50  0000 C CNN
 	1    2700 2550
@@
 F 0 "D8" H 3400 2650 50  0000 C CNN
 F 1 "D" H 3400 2450 50  0001 C CNN
-F 2 "Keyboard:DIODE" H 3400 2550 50  0001 C CNN
+F 2 "Diodes_SMD:SOD-123" H 3400 2550 50  0001 C CNN
 F 3 "" H 3400 2550 50  0000 C CNN
 	1    3400 2550
@@
 F 0 "SW12" H 3550 3410 50  0000 C CNN
 F 1 "PLUS" V 3400 3220 50  0000 C CNN
-F 2 "Keyboard:CHERRY_PLATE_100H" H 3400 3300 50  0001 C CNN
+F 2 "Keyboard:CHERRY_PLATE_200V" H 3400 3300 50  0001 C CNN
 F 3 "" H 3400 3300 50  0000 C CNN
 	1    3400 3300
@@
 F 0 "D9" H 1300 3850 50  0000 C CNN
 F 1 "D" H 1300 3650 50  0001 C CNN
-F 2 "Keyboard:DIODE" H 1300 3750 50  0001 C CNN
+F 2 "Diodes_SMD:SOD-123" H 1300 3750 50  0001 C CNN
 F 3 "" H 1300 3750 50  0000 C CNN
 	1    1300 3750
@@
 F 0 "D10" H 2000 3850 50  0000 C CNN
 F 1 "D" H 2000 3650 50  0001 C CNN
-F 2 "Keyboard:DIODE" H 2000 3750 50  0001 C CNN
+F 2 "Diodes_SMD:SOD-123" H 2000 3750 50  0001 C CNN
 F 3 "" H 2000 3750 50  0000 C CNN
 	1    2000 3750
@@
 F 0 "D11" H 2700 3850 50  0000 C CNN
 F 1 "D" H 2700 3650 50  0001 C CNN
-F 2 "Keyboard:DIODE" H 2700 3750 50  0001 C CNN
+F 2 "Diodes_SMD:SOD-123" H 2700 3750 50  0001 C CNN
 F 3 "" H 2700 3750 50  0000 C CNN
 	1    2700 3750
@@
 F 0 "D12" H 3400 3850 50  0000 C CNN
 F 1 "D" H 3400 3650 50  0001 C CNN
-F 2 "Keyboard:DIODE" H 3400 3750 50  0001 C CNN
+F 2 "Diodes_SMD:SOD-123" H 3400 3750 50  0001 C CNN
 F 3 "" H 3400 3750 50  0000 C CNN
 	1    3400 3750
@@
 F 0 "SW16" H 3550 4610 50  0000 C CNN
 F 1 "ENTER" V 3400 4420 50  0000 C CNN
-F 2 "Keyboard:CHERRY_PLATE_100H" H 3400 4500 50  0001 C CNN
+F 2 "Keyboard:CHERRY_PLATE_200V" H 3400 4500 50  0001 C CNN
 F 3 "" H 3400 4500 50  0000 C CNN
 	1    3400 4500
@@
 F 0 "D13" H 1300 5050 50  0000 C CNN
 F 1 "D" H 1300 4850 50  0001 C CNN
-F 2 "Keyboard:DIODE" H 1300 4950 50  0001 C CNN
+F 2 "Diodes_SMD:SOD-123" H 1300 4950 50  0001 C CNN
 F 3 "" H 1300 4950 50  0000 C CNN
 	1    1300 4950
@@
 F 0 "D14" H 2000 5050 50  0000 C CNN
 F 1 "D" H 2000 4850 50  0001 C CNN
-F 2 "Keyboard:DIODE" H 2000 4950 50  0001 C CNN
+F 2 "Diodes_SMD:SOD-123" H 2000 4950 50  0001 C CNN
 F 3 "" H 2000 4950 50  0000 C CNN
 	1    2000 4950
@@
 F 0 "D15" H 2700 5050 50  0000 C CNN
 F 1 "D" H 2700 4850 50  0001 C CNN
-F 2 "Keyboard:DIODE" H 2700 4950 50  0001 C CNN
+F 2 "Diodes_SMD:SOD-123" H 2700 4950 50  0001 C CNN
 F 3 "" H 2700 4950 50  0000 C CNN
 	1    2700 4950
@@
 F 0 "D16" H 3400 5050 50  0000 C CNN
 F 1 "D" H 3400 4850 50  0001 C CNN
-F 2 "Keyboard:DIODE" H 3400 4950 50  0001 C CNN
+F 2 "Diodes_SMD:SOD-123" H 3400 4950 50  0001 C CNN
 F 3 "" H 3400 4950 50  0000 C CNN
 	1    3400 4950
@@
 F 0 "SW20" H 3550 5710 50  0000 C CNN
 F 1 "0" V 3400 5520 50  0000 C CNN
-F 2 "Keyboard:CHERRY_PLATE_100H" H 3400 5600 50  0001 C CNN
+F 2 "Keyboard:CHERRY_PLATE_200H" H 3400 5600 50  0001 C CNN
 F 3 "" H 3400 5600 50  0000 C CNN
 	1    3400 5600
@@
 F 0 "D17" H 1300 6150 50  0000 C CNN
 F 1 "D" H 1300 5950 50  0001 C CNN
-F 2 "Keyboard:DIODE" H 1300 6050 50  0001 C CNN
+F 2 "Diodes_SMD:SOD-123" H 1300 6050 50  0001 C CNN
 F 3 "" H 1300 6050 50  0000 C CNN
 	1    1300 6050
@@
 F 0 "D18" H 2000 6150 50  0000 C CNN
 F 1 "D" H 2000 5950 50  0001 C CNN
-F 2 "Keyboard:DIODE" H 2000 6050 50  0001 C CNN
+F 2 "Diodes_SMD:SOD-123" H 2000 6050 50  0001 C CNN
 F 3 "" H 2000 6050 50  0000 C CNN
 	1    2000 6050
@@
 F 0 "D19" H 2700 6150 50  0000 C CNN
 F 1 "D" H 2700 5950 50  0001 C CNN
-F 2 "Keyboard:DIODE" H 2700 6050 50  0001 C CNN
+F 2 "Diodes_SMD:SOD-123" H 2700 6050 50  0001 C CNN
 F 3 "" H 2700 6050 50  0000 C CNN
 	1    2700 6050
@@
 F 0 "D20" H 3400 6150 50  0000 C CNN
 F 1 "D" H 3400 5950 50  0001 C CNN
-F 2 "Keyboard:DIODE" H 3400 6050 50  0001 C CNN
+F 2 "Diodes_SMD:SOD-123" H 3400 6050 50  0001 C CNN
 F 3 "" H 3400 6050 50  0000 C CNN
 	1    3400 6050
@@
 F 0 "D21" H 4100 6150 50  0000 C CNN
 F 1 "D" H 4100 5950 50  0001 C CNN
-F 2 "Keyboard:DIODE" H 4100 6050 50  0001 C CNN
+F 2 "Diodes_SMD:SOD-123" H 4100 6050 50  0001 C CNN
 F 3 "" H 4100 6050 50  0000 C CNN
 	1    4100 6050
@@
 F 0 "D22" H 8050 6250 50  0000 C CNN
 F 1 "LED" H 8050 6050 50  0000 C CNN
-F 2 "Keyboard:LED_3MM" H 8050 6150 50  0001 C CNN
+F 2 "Keyboard:CHERRY_MX_LED" H 8050 6150 50  0001 C CNN
 F 3 "" H 8050 6150 50  0000 C CNN
 	1    8050 6150
@@
 Text Label 5650 4850 2    60   ~ 0
 XTAL1
-Text Label 6450 4850 0    60   ~ 0
+Text Label 6550 4850 0    60   ~ 0
 XTAL2
 $Comp
@@
 L C C3
 U 1 1 57D6B38B
-P 6450 5150
-F 0 "C3" H 6475 5250 50  0000 L CNN
-F 1 "18p" H 6475 5050 50  0000 L CNN
-F 2 "Keyboard:C_0805" H 6488 5000 50  0001 C CNN
-F 3 "" H 6450 5150 50  0000 C CNN
-	1    6450 5150
-	1    0    0    -1
-$EndComp
-$Comp
-L Crystal Y1
-U 1 1 57D6B47F
-P 6050 4850
-F 0 "Y1" H 6050 5000 50  0000 C CNN
-F 1 "16MHz" H 6050 4700 50  0000 C CNN
-F 2 "Crystals:Crystal_HC49-U_Vertical" H 6050 4850 50  0001 C CNN
-F 3 "" H 6050 4850 50  0000 C CNN
-	1    6050 4850
+P 6550 5150
+F 0 "C3" H 6575 5250 50  0000 L CNN
+F 1 "18p" H 6575 5050 50  0000 L CNN
+F 2 "Keyboard:C_0805" H 6588 5000 50  0001 C CNN
+F 3 "" H 6550 5150 50  0000 C CNN
+	1    6550 5150
 	1    0    0    -1
 $EndComp
@@
 L GND #PWR06
 U 1 1 57D6B69A
-P 6450 5400
-F 0 "#PWR06" H 6450 5150 50  0001 C CNN
-F 1 "GND" H 6450 5250 50  0000 C CNN
-F 2 "" H 6450 5400 50  0000 C CNN
-F 3 "" H 6450 5400 50  0000 C CNN
-	1    6450 5400
+P 6550 5400
+F 0 "#PWR06" H 6550 5150 50  0001 C CNN
+F 1 "GND" H 6550 5250 50  0000 C CNN
+F 2 "" H 6550 5400 50  0000 C CNN
+F 3 "" H 6550 5400 50  0000 C CNN
+	1    6550 5400
 	1    0    0    -1
 $EndComp
@@
 $EndComp
 $Comp
-L +5V #PWR012
+L +5V #PWR09
 U 1 1 57D75692
 P 10000 5000
-F 0 "#PWR012" H 10000 4850 50  0001 C CNN
+F 0 "#PWR09" H 10000 4850 50  0001 C CNN
 F 1 "+5V" H 10000 5140 50  0000 C CNN
 F 2 "" H 10000 5000 50  0000 C CNN
@@
 $EndComp
 $Comp
-L GND #PWR013
+L GND #PWR010
 U 1 1 57D75718
 P 10000 5600
-F 0 "#PWR013" H 10000 5350 50  0001 C CNN
+F 0 "#PWR010" H 10000 5350 50  0001 C CNN
 F 1 "GND" H 10000 5450 50  0000 C CNN
 F 2 "" H 10000 5600 50  0000 C CNN
@@
 	4400 6200 4400 6600
 Wire Wire Line
-	6200 4850 6450 4850
-Wire Wire Line
-	6450 4850 6450 5000
-Wire Wire Line
-	6450 5300 6450 5400
+	6300 4850 6550 4850
+Wire Wire Line
+	6550 4850 6550 5000
+Wire Wire Line
+	6550 5300 6550 5400
 Wire Wire Line
 	5900 4850 5650 4850
@@
 Connection ~ 10000 5600
 $Comp
-L VCC #PWR?
+L VCC #PWR011
 U 1 1 583F89D3
 P 9800 5000
-F 0 "#PWR?" H 9800 4850 50  0001 C CNN
+F 0 "#PWR011" H 9800 4850 50  0001 C CNN
 F 1 "VCC" H 9800 5150 50  0000 C CNN
 F 2 "" H 9800 5000 50  0000 C CNN
@@
 $EndComp
 $Comp
-L +5V #PWR?
+L +5V #PWR012
 U 1 1 583FB50A
 P 5850 1700
-F 0 "#PWR?" H 5850 1550 50  0001 C CNN
+F 0 "#PWR012" H 5850 1550 50  0001 C CNN
 F 1 "+5V" H 5850 1840 50  0000 C CNN
 F 2 "" H 5850 1700 50  0000 C CNN
@@
 	5700 1500 5700 1000
 $Comp
-L VCC #PWR?
+L VCC #PWR013
 U 1 1 583FB754
 P 5700 1000
-F 0 "#PWR?" H 5700 850 50  0001 C CNN
+F 0 "#PWR013" H 5700 850 50  0001 C CNN
 F 1 "VCC" H 5700 1150 50  0000 C CNN
 F 2 "" H 5700 1000 50  0000 C CNN
@@
 $EndComp
 $Comp
-L VCC #PWR?
+L VCC #PWR014
 U 1 1 583FE193
 P 6050 2700
-F 0 "#PWR?" H 6050 2550 50  0001 C CNN
+F 0 "#PWR014" H 6050 2550 50  0001 C CNN
 F 1 "VCC" H 6050 2850 50  0000 C CNN
 F 2 "" H 6050 2700 50  0000 C CNN
@@
 F 0 "SW22" H 8000 4960 50  0000 C CNN
 F 1 "SW_PUSH" H 7850 4770 50  0000 C CNN
-F 2 "" H 7850 4850 50  0000 C CNN
+F 2 "Buttons_Switches_SMD:SW_SPST_B3S-1000" H 7850 4850 50  0001 C CNN
 F 3 "" H 7850 4850 50  0000 C CNN
 	1    7850 4850
@@
 $EndComp
 $Comp
-L GND #PWR?
+L GND #PWR015
 U 1 1 583FE5A3
 P 8150 4850
-F 0 "#PWR?" H 8150 4600 50  0001 C CNN
+F 0 "#PWR015" H 8150 4600 50  0001 C CNN
 F 1 "GND" H 8150 4700 50  0000 C CNN
 F 2 "" H 8150 4850 50  0000 C CNN
@@
 	1    0    0    -1
 $EndComp
+$Comp
+L CRYSTAL_SMD X1
+U 1 1 583F85A8
+P 6100 4850
+F 0 "X1" H 6100 4940 50  0000 C CNN
+F 1 "16MHz" H 6130 4740 50  0000 L CNN
+F 2 "Crystals:Crystal_SMD_5032_4Pads" H 6100 4850 50  0001 C CNN
+F 3 "" H 6100 4850 50  0000 C CNN
+	1    6100 4850
+	1    0    0    -1
+$EndComp
+$Comp
+L GND #PWR016
+U 1 1 583F8B57
+P 6100 4950
+F 0 "#PWR016" H 6100 4700 50  0001 C CNN
+F 1 "GND" H 6100 4800 50  0000 C CNN
+F 2 "" H 6100 4950 50  0000 C CNN
+F 3 "" H 6100 4950 50  0000 C CNN
+	1    6100 4950
+	1    0    0    -1
+$EndComp

Commit message: Add SMD micro USB B, move MCU
Parts:
- P1: footprint Connect:USB_Micro-B -> 10118192-0001LF:10118192-0001LF
Changed lines of the file:
@@
 LIBS:contrib
 LIBS:valves
+LIBS:10118192-0001LF
 LIBS:Numpad-cache
 EELAYER 25 0
@@
 F 0 "P1" H 5025 1675 50  0000 C CNN
 F 1 "USB-MICRO-B" H 4700 2000 50  0000 C CNN
-F 2 "Connect:USB_Micro-B" V 4650 1700 50  0001 C CNN
+F 2 "10118192-0001LF:10118192-0001LF" V 4650 1700 50  0001 C CNN
 F 3 "" V 4650 1700 50  0000 C CNN
 	1    4700 1800

Commit message: Add mounting holes to schematic
Parts:
- added P1, P2, P3, P4: HOLE, symbol CONN_01X01
Connections:
- net GND: now also P1.1 (P1), P2.1 (P1), P3.1 (P1), P4.1 (P1)
Changed lines of the file:
@@
 	1    0    0    -1
 $EndComp
+$Comp
+L CONN_01X01 P1
+U 1 1 5840D1D0
+P 9650 3150
+F 0 "P1" H 9650 3250 50  0000 C CNN
+F 1 "HOLE" V 9750 3150 50  0000 C CNN
+F 2 "" H 9650 3150 50  0000 C CNN
+F 3 "" H 9650 3150 50  0000 C CNN
+	1    9650 3150
+	1    0    0    -1
+$EndComp
+$Comp
+L CONN_01X01 P2
+U 1 1 5840D324
+P 9650 3400
+F 0 "P2" H 9650 3500 50  0000 C CNN
+F 1 "HOLE" V 9750 3400 50  0000 C CNN
+F 2 "" H 9650 3400 50  0000 C CNN
+F 3 "" H 9650 3400 50  0000 C CNN
+	1    9650 3400
+	1    0    0    -1
+$EndComp
+$Comp
+L CONN_01X01 P3
+U 1 1 5840D3EB
+P 9650 3650
+F 0 "P3" H 9650 3750 50  0000 C CNN
+F 1 "HOLE" V 9750 3650 50  0000 C CNN
+F 2 "" H 9650 3650 50  0000 C CNN
+F 3 "" H 9650 3650 50  0000 C CNN
+	1    9650 3650
+	1    0    0    -1
+$EndComp
+$Comp
+L CONN_01X01 P4
+U 1 1 5840D4B5
+P 9650 3900
+F 0 "P4" H 9650 4000 50  0000 C CNN
+F 1 "HOLE" V 9750 3900 50  0000 C CNN
+F 2 "" H 9650 3900 50  0000 C CNN
+F 3 "" H 9650 3900 50  0000 C CNN
+	1    9650 3900
+	1    0    0    -1
+$EndComp
+$Comp
+L GND #PWR?
+U 1 1 5840D946
+P 9450 3900
+F 0 "#PWR?" H 9450 3650 50  0001 C CNN
+F 1 "GND" H 9450 3750 50  0000 C CNN
+F 2 "" H 9450 3900 50  0000 C CNN
+F 3 "" H 9450 3900 50  0000 C CNN
+	1    9450 3900
+	1    0    0    -1
+$EndComp
+Wire Wire Line
+	9450 3150 9450 3900
+Connection ~ 9450 3400
+Connection ~ 9450 3650
 $EndSCHEMATC
