File: pcb/Numpad.sch (KiCad schematic (older format))
At the start: 61 parts, among them P1 HOLE, P1 USB-MICRO-B, P2 HOLE, P3 HOLE, P4 HOLE, SW1 F1, SW10 8, SW11 9, SW12 PLUS, SW13 4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

Commit message: Fix mounting hole names
Parts:
- renumbered P1 to P2, P2 to P3, P3 to P4, P4 to P5
Changed lines of the file:
@@
 $EndComp
 $Comp
-L GND #PWR01
+L GND #PWR1
 U 1 1 57D6027E
 P 4850 1100
-F 0 "#PWR01" H 4850 850 50  0001 C CNN
+F 0 "#PWR1" H 4850 850 50  0001 C CNN
 F 1 "GND" H 4850 950 50  0000 C CNN
 F 2 "" H 4850 1100 50  0000 C CNN
@@
 $EndComp
 $Comp
-L +5V #PWR02
+L +5V #PWR2
 U 1 1 57D602D0
 P 5100 2300
-F 0 "#PWR02" H 5100 2150 50  0001 C CNN
+F 0 "#PWR2" H 5100 2150 50  0001 C CNN
 F 1 "+5V" H 5100 2440 50  0000 C CNN
 F 2 "" H 5100 2300 50  0000 C CNN
@@
 COL4
 $Comp
-L GND #PWR03
+L GND #PWR3
 U 1 1 57D60904
 P 5350 2900
-F 0 "#PWR03" H 5350 2650 50  0001 C CNN
+F 0 "#PWR3" H 5350 2650 50  0001 C CNN
 F 1 "GND" H 5350 2750 50  0000 C CNN
 F 2 "" H 5350 2900 50  0000 C CNN
@@
 $EndComp
 $Comp
-L GND #PWR04
+L GND #PWR13
 U 1 1 57D6A2D0
 P 8250 6150
-F 0 "#PWR04" H 8250 5900 50  0001 C CNN
+F 0 "#PWR13" H 8250 5900 50  0001 C CNN
 F 1 "GND" H 8250 6000 50  0000 C CNN
 F 2 "" H 8250 6150 50  0000 C CNN
@@
 $EndComp
 $Comp
-L GND #PWR05
+L GND #PWR4
 U 1 1 57D6B61E
 P 5650 5400
-F 0 "#PWR05" H 5650 5150 50  0001 C CNN
+F 0 "#PWR4" H 5650 5150 50  0001 C CNN
 F 1 "GND" H 5650 5250 50  0000 C CNN
 F 2 "" H 5650 5400 50  0000 C CNN
@@
 $EndComp
 $Comp
-L GND #PWR06
+L GND #PWR11
 U 1 1 57D6B69A
 P 6550 5400
-F 0 "#PWR06" H 6550 5150 50  0001 C CNN
+F 0 "#PWR11" H 6550 5150 50  0001 C CNN
 F 1 "GND" H 6550 5250 50  0000 C CNN
 F 2 "" H 6550 5400 50  0000 C CNN
@@
 $EndComp
 $Comp
-L GND #PWR07
+L GND #PWR6
 U 1 1 57D6BCA7
 P 5700 4000
-F 0 "#PWR07" H 5700 3750 50  0001 C CNN
+F 0 "#PWR6" H 5700 3750 50  0001 C CNN
 F 1 "GND" H 5700 3850 50  0000 C CNN
 F 2 "" H 5700 4000 50  0000 C CNN
@@
 ISP_RESET
 $Comp
-L +5V #PWR08
+L +5V #PWR7
 U 1 1 57D6C60C
 P 5850 1000
-F 0 "#PWR08" H 5850 850 50  0001 C CNN
+F 0 "#PWR7" H 5850 850 50  0001 C CNN
 F 1 "+5V" H 5850 1140 50  0000 C CNN
 F 2 "" H 5850 1000 50  0000 C CNN
@@
 $EndComp
 $Comp
-L +5V #PWR09
+L +5V #PWR16
 U 1 1 57D75692
 P 10000 5000
-F 0 "#PWR09" H 10000 4850 50  0001 C CNN
+F 0 "#PWR16" H 10000 4850 50  0001 C CNN
 F 1 "+5V" H 10000 5140 50  0000 C CNN
 F 2 "" H 10000 5000 50  0000 C CNN
@@
 $EndComp
 $Comp
-L GND #PWR010
+L GND #PWR17
 U 1 1 57D75718
 P 10000 5600
-F 0 "#PWR010" H 10000 5350 50  0001 C CNN
+F 0 "#PWR17" H 10000 5350 50  0001 C CNN
 F 1 "GND" H 10000 5450 50  0000 C CNN
 F 2 "" H 10000 5600 50  0000 C CNN
@@
 Connection ~ 10000 5600
 $Comp
-L VCC #PWR011
+L VCC #PWR15
 U 1 1 583F89D3
 P 9800 5000
-F 0 "#PWR011" H 9800 4850 50  0001 C CNN
+F 0 "#PWR15" H 9800 4850 50  0001 C CNN
 F 1 "VCC" H 9800 5150 50  0000 C CNN
 F 2 "" H 9800 5000 50  0000 C CNN
@@
 $EndComp
 $Comp
-L +5V #PWR012
+L +5V #PWR8
 U 1 1 583FB50A
 P 5850 1700
-F 0 "#PWR012" H 5850 1550 50  0001 C CNN
+F 0 "#PWR8" H 5850 1550 50  0001 C CNN
 F 1 "+5V" H 5850 1840 50  0000 C CNN
 F 2 "" H 5850 1700 50  0000 C CNN
@@
 	5700 1500 5700 1000
 $Comp
-L VCC #PWR013
+L VCC #PWR5
 U 1 1 583FB754
 P 5700 1000
-F 0 "#PWR013" H 5700 850 50  0001 C CNN
+F 0 "#PWR5" H 5700 850 50  0001 C CNN
 F 1 "VCC" H 5700 1150 50  0000 C CNN
 F 2 "" H 5700 1000 50  0000 C CNN
@@
 $EndComp
 $Comp
-L VCC #PWR014
+L VCC #PWR9
 U 1 1 583FE193
 P 6050 2700
-F 0 "#PWR014" H 6050 2550 50  0001 C CNN
+F 0 "#PWR9" H 6050 2550 50  0001 C CNN
 F 1 "VCC" H 6050 2850 50  0000 C CNN
 F 2 "" H 6050 2700 50  0000 C CNN
@@
 $EndComp
 $Comp
-L GND #PWR015
+L GND #PWR12
 U 1 1 583FE5A3
 P 8150 4850
-F 0 "#PWR015" H 8150 4600 50  0001 C CNN
+F 0 "#PWR12" H 8150 4600 50  0001 C CNN
 F 1 "GND" H 8150 4700 50  0000 C CNN
 F 2 "" H 8150 4850 50  0000 C CNN
@@
 $EndComp
 $Comp
-L GND #PWR016
+L GND #PWR10
 U 1 1 583F8B57
 P 6100 4950
-F 0 "#PWR016" H 6100 4700 50  0001 C CNN
+F 0 "#PWR10" H 6100 4700 50  0001 C CNN
 F 1 "GND" H 6100 4800 50  0000 C CNN
 F 2 "" H 6100 4950 50  0000 C CNN
@@
 $EndComp
 $Comp
-L CONN_01X01 P1
+L CONN_01X01 P2
 U 1 1 5840D1D0
 P 9650 3150
-F 0 "P1" H 9650 3250 50  0000 C CNN
+F 0 "P2" H 9650 3250 50  0000 C CNN
 F 1 "HOLE" V 9750 3150 50  0000 C CNN
 F 2 "" H 9650 3150 50  0000 C CNN
@@
 $EndComp
 $Comp
-L CONN_01X01 P2
+L CONN_01X01 P3
 U 1 1 5840D324
 P 9650 3400
-F 0 "P2" H 9650 3500 50  0000 C CNN
+F 0 "P3" H 9650 3500 50  0000 C CNN
 F 1 "HOLE" V 9750 3400 50  0000 C CNN
 F 2 "" H 9650 3400 50  0000 C CNN
@@
 $EndComp
 $Comp
-L CONN_01X01 P3
+L CONN_01X01 P4
 U 1 1 5840D3EB
 P 9650 3650
-F 0 "P3" H 9650 3750 50  0000 C CNN
+F 0 "P4" H 9650 3750 50  0000 C CNN
 F 1 "HOLE" V 9750 3650 50  0000 C CNN
 F 2 "" H 9650 3650 50  0000 C CNN
@@
 $EndComp
 $Comp
-L CONN_01X01 P4
+L CONN_01X01 P5
 U 1 1 5840D4B5
 P 9650 3900
-F 0 "P4" H 9650 4000 50  0000 C CNN
+F 0 "P5" H 9650 4000 50  0000 C CNN
 F 1 "HOLE" V 9750 3900 50  0000 C CNN
 F 2 "" H 9650 3900 50  0000 C CNN
@@
 $EndComp
 $Comp
-L GND #PWR?
+L GND #PWR14
 U 1 1 5840D946
 P 9450 3900
-F 0 "#PWR?" H 9450 3650 50  0001 C CNN
+F 0 "#PWR14" H 9450 3650 50  0001 C CNN
 F 1 "GND" H 9450 3750 50  0000 C CNN
 F 2 "" H 9450 3900 50  0000 C CNN

Commit message: Associate holes with footprints
Parts:
- P2, P3, P4, P5: footprint (none) -> Connect:1pin
Changed lines of the file:
@@
 $EndComp
 $Comp
-L GND #PWR1
+L GND #PWR01
 U 1 1 57D6027E
 P 4850 1100
-F 0 "#PWR1" H 4850 850 50  0001 C CNN
+F 0 "#PWR01" H 4850 850 50  0001 C CNN
 F 1 "GND" H 4850 950 50  0000 C CNN
 F 2 "" H 4850 1100 50  0000 C CNN
@@
 $EndComp
 $Comp
-L +5V #PWR2
+L +5V #PWR02
 U 1 1 57D602D0
 P 5100 2300
-F 0 "#PWR2" H 5100 2150 50  0001 C CNN
+F 0 "#PWR02" H 5100 2150 50  0001 C CNN
 F 1 "+5V" H 5100 2440 50  0000 C CNN
 F 2 "" H 5100 2300 50  0000 C CNN
@@
 COL4
 $Comp
-L GND #PWR3
+L GND #PWR03
 U 1 1 57D60904
 P 5350 2900
-F 0 "#PWR3" H 5350 2650 50  0001 C CNN
+F 0 "#PWR03" H 5350 2650 50  0001 C CNN
 F 1 "GND" H 5350 2750 50  0000 C CNN
 F 2 "" H 5350 2900 50  0000 C CNN
@@
 $EndComp
 $Comp
-L GND #PWR13
+L GND #PWR04
 U 1 1 57D6A2D0
 P 8250 6150
-F 0 "#PWR13" H 8250 5900 50  0001 C CNN
+F 0 "#PWR04" H 8250 5900 50  0001 C CNN
 F 1 "GND" H 8250 6000 50  0000 C CNN
 F 2 "" H 8250 6150 50  0000 C CNN
@@
 $EndComp
 $Comp
-L GND #PWR4
+L GND #PWR05
 U 1 1 57D6B61E
 P 5650 5400
-F 0 "#PWR4" H 5650 5150 50  0001 C CNN
+F 0 "#PWR05" H 5650 5150 50  0001 C CNN
 F 1 "GND" H 5650 5250 50  0000 C CNN
 F 2 "" H 5650 5400 50  0000 C CNN
@@
 $EndComp
 $Comp
-L GND #PWR11
+L GND #PWR06
 U 1 1 57D6B69A
 P 6550 5400
-F 0 "#PWR11" H 6550 5150 50  0001 C CNN
+F 0 "#PWR06" H 6550 5150 50  0001 C CNN
 F 1 "GND" H 6550 5250 50  0000 C CNN
 F 2 "" H 6550 5400 50  0000 C CNN
@@
 $EndComp
 $Comp
-L GND #PWR6
+L GND #PWR07
 U 1 1 57D6BCA7
 P 5700 4000
-F 0 "#PWR6" H 5700 3750 50  0001 C CNN
+F 0 "#PWR07" H 5700 3750 50  0001 C CNN
 F 1 "GND" H 5700 3850 50  0000 C CNN
 F 2 "" H 5700 4000 50  0000 C CNN
@@
 ISP_RESET
 $Comp
-L +5V #PWR7
+L +5V #PWR08
 U 1 1 57D6C60C
 P 5850 1000
-F 0 "#PWR7" H 5850 850 50  0001 C CNN
+F 0 "#PWR08" H 5850 850 50  0001 C CNN
 F 1 "+5V" H 5850 1140 50  0000 C CNN
 F 2 "" H 5850 1000 50  0000 C CNN
@@
 $EndComp
 $Comp
-L +5V #PWR16
+L +5V #PWR09
 U 1 1 57D75692
 P 10000 5000
-F 0 "#PWR16" H 10000 4850 50  0001 C CNN
+F 0 "#PWR09" H 10000 4850 50  0001 C CNN
 F 1 "+5V" H 10000 5140 50  0000 C CNN
 F 2 "" H 10000 5000 50  0000 C CNN
@@
 $EndComp
 $Comp
-L GND #PWR17
+L GND #PWR010
 U 1 1 57D75718
 P 10000 5600
-F 0 "#PWR17" H 10000 5350 50  0001 C CNN
+F 0 "#PWR010" H 10000 5350 50  0001 C CNN
 F 1 "GND" H 10000 5450 50  0000 C CNN
 F 2 "" H 10000 5600 50  0000 C CNN
@@
 Connection ~ 10000 5600
 $Comp
-L VCC #PWR15
+L VCC #PWR011
 U 1 1 583F89D3
 P 9800 5000
-F 0 "#PWR15" H 9800 4850 50  0001 C CNN
+F 0 "#PWR011" H 9800 4850 50  0001 C CNN
 F 1 "VCC" H 9800 5150 50  0000 C CNN
 F 2 "" H 9800 5000 50  0000 C CNN
@@
 $EndComp
 $Comp
-L +5V #PWR8
+L +5V #PWR012
 U 1 1 583FB50A
 P 5850 1700
-F 0 "#PWR8" H 5850 1550 50  0001 C CNN
+F 0 "#PWR012" H 5850 1550 50  0001 C CNN
 F 1 "+5V" H 5850 1840 50  0000 C CNN
 F 2 "" H 5850 1700 50  0000 C CNN
@@
 	5700 1500 5700 1000
 $Comp
-L VCC #PWR5
+L VCC #PWR013
 U 1 1 583FB754
 P 5700 1000
-F 0 "#PWR5" H 5700 850 50  0001 C CNN
+F 0 "#PWR013" H 5700 850 50  0001 C CNN
 F 1 "VCC" H 5700 1150 50  0000 C CNN
 F 2 "" H 5700 1000 50  0000 C CNN
@@
 $EndComp
 $Comp
-L VCC #PWR9
+L VCC #PWR014
 U 1 1 583FE193
 P 6050 2700
-F 0 "#PWR9" H 6050 2550 50  0001 C CNN
+F 0 "#PWR014" H 6050 2550 50  0001 C CNN
 F 1 "VCC" H 6050 2850 50  0000 C CNN
 F 2 "" H 6050 2700 50  0000 C CNN
@@
 $EndComp
 $Comp
-L GND #PWR12
+L GND #PWR015
 U 1 1 583FE5A3
 P 8150 4850
-F 0 "#PWR12" H 8150 4600 50  0001 C CNN
+F 0 "#PWR015" H 8150 4600 50  0001 C CNN
 F 1 "GND" H 8150 4700 50  0000 C CNN
 F 2 "" H 8150 4850 50  0000 C CNN
@@
 $EndComp
 $Comp
-L GND #PWR10
+L GND #PWR016
 U 1 1 583F8B57
 P 6100 4950
-F 0 "#PWR10" H 6100 4700 50  0001 C CNN
+F 0 "#PWR016" H 6100 4700 50  0001 C CNN
 F 1 "GND" H 6100 4800 50  0000 C CNN
 F 2 "" H 6100 4950 50  0000 C CNN
@@
 F 0 "P2" H 9650 3250 50  0000 C CNN
 F 1 "HOLE" V 9750 3150 50  0000 C CNN
-F 2 "" H 9650 3150 50  0000 C CNN
+F 2 "Connect:1pin" H 9650 3150 50  0001 C CNN
 F 3 "" H 9650 3150 50  0000 C CNN
 	1    9650 3150
@@
 F 0 "P3" H 9650 3500 50  0000 C CNN
 F 1 "HOLE" V 9750 3400 50  0000 C CNN
-F 2 "" H 9650 3400 50  0000 C CNN
+F 2 "Connect:1pin" H 9650 3400 50  0001 C CNN
 F 3 "" H 9650 3400 50  0000 C CNN
 	1    9650 3400
@@
 F 0 "P4" H 9650 3750 50  0000 C CNN
 F 1 "HOLE" V 9750 3650 50  0000 C CNN
-F 2 "" H 9650 3650 50  0000 C CNN
+F 2 "Connect:1pin" H 9650 3650 50  0001 C CNN
 F 3 "" H 9650 3650 50  0000 C CNN
 	1    9650 3650
@@
 F 0 "P5" H 9650 4000 50  0000 C CNN
 F 1 "HOLE" V 9750 3900 50  0000 C CNN
-F 2 "" H 9650 3900 50  0000 C CNN
+F 2 "Connect:1pin" H 9650 3900 50  0001 C CNN
 F 3 "" H 9650 3900 50  0000 C CNN
 	1    9650 3900
@@
 $EndComp
 $Comp
-L GND #PWR14
+L GND #PWR017
 U 1 1 5840D946
 P 9450 3900
-F 0 "#PWR14" H 9450 3650 50  0001 C CNN
+F 0 "#PWR017" H 9450 3650 50  0001 C CNN
 F 1 "GND" H 9450 3750 50  0000 C CNN
 F 2 "" H 9450 3900 50  0000 C CNN

Commit message: Add my own key footprints
Parts:
- SW1: value F1 -> F13; footprint Keyboard:CHERRY_PLATE_100H -> Tim's Cherry MX:CHERRY_PLATE_100H
- SW10, SW11, SW13, SW14, SW15, SW17, SW18, SW19, SW21, SW5, SW6, SW7, SW8, SW9: footprint Keyboard:CHERRY_PLATE_100H -> Tim's Cherry MX:CHERRY_PLATE_100H
- SW12, SW16: footprint Keyboard:CHERRY_PLATE_200V -> Tim's Cherry MX:CHERRY_PLATE_200V
- SW2: value F2 -> F14; footprint Keyboard:CHERRY_PLATE_100H -> Tim's Cherry MX:CHERRY_PLATE_100H
- SW20: footprint Keyboard:CHERRY_PLATE_200H -> Tim's Cherry MX:CHERRY_PLATE_200H
- SW3: value F3 -> F15; footprint Keyboard:CHERRY_PLATE_100H -> Tim's Cherry MX:CHERRY_PLATE_100H
- SW4: value F4 -> F16; footprint Keyboard:CHERRY_PLATE_100H -> Tim's Cherry MX:CHERRY_PLATE_100H
Changed lines of the file:
@@
 P 1300 900
 F 0 "SW1" H 1450 1010 50  0000 C CNN
-F 1 "F1" V 1300 820 50  0000 C CNN
-F 2 "Keyboard:CHERRY_PLATE_100H" H 1300 900 50  0001 C CNN
+F 1 "F13" V 1300 820 50  0000 C CNN
+F 2 "Tim's Cherry MX:CHERRY_PLATE_100H" H 1300 900 50  0001 C CNN
 F 3 "" H 1300 900 50  0000 C CNN
 	1    1300 900
@@
 P 2700 900
 F 0 "SW3" H 2850 1010 50  0000 C CNN
-F 1 "F3" V 2700 820 50  0000 C CNN
-F 2 "Keyboard:CHERRY_PLATE_100H" H 2700 900 50  0001 C CNN
+F 1 "F15" V 2700 820 50  0000 C CNN
+F 2 "Tim's Cherry MX:CHERRY_PLATE_100H" H 2700 900 50  0001 C CNN
 F 3 "" H 2700 900 50  0000 C CNN
 	1    2700 900
@@
 P 3400 900
 F 0 "SW4" H 3550 1010 50  0000 C CNN
-F 1 "F4" V 3400 820 50  0000 C CNN
-F 2 "Keyboard:CHERRY_PLATE_100H" H 3400 900 50  0001 C CNN
+F 1 "F16" V 3400 820 50  0000 C CNN
+F 2 "Tim's Cherry MX:CHERRY_PLATE_100H" H 3400 900 50  0001 C CNN
 F 3 "" H 3400 900 50  0000 C CNN
 	1    3400 900
@@
 P 2000 900
 F 0 "SW2" H 2150 1010 50  0000 C CNN
-F 1 "F2" V 2000 820 50  0000 C CNN
-F 2 "Keyboard:CHERRY_PLATE_100H" H 2000 900 50  0001 C CNN
+F 1 "F14" V 2000 820 50  0000 C CNN
+F 2 "Tim's Cherry MX:CHERRY_PLATE_100H" H 2000 900 50  0001 C CNN
 F 3 "" H 2000 900 50  0000 C CNN
 	1    2000 900
@@
 F 0 "SW5" H 1450 2210 50  0000 C CNN
 F 1 "NUMLOCK" H 1300 2020 50  0000 C CNN
-F 2 "Keyboard:CHERRY_PLATE_100H" H 1300 2100 50  0001 C CNN
+F 2 "Tim's Cherry MX:CHERRY_PLATE_100H" H 1300 2100 50  0001 C CNN
 F 3 "" H 1300 2100 50  0000 C CNN
 	1    1300 2100
@@
 F 0 "SW7" H 2850 2210 50  0000 C CNN
 F 1 "STAR" V 2700 2020 50  0000 C CNN
-F 2 "Keyboard:CHERRY_PLATE_100H" H 2700 2100 50  0001 C CNN
+F 2 "Tim's Cherry MX:CHERRY_PLATE_100H" H 2700 2100 50  0001 C CNN
 F 3 "" H 2700 2100 50  0000 C CNN
 	1    2700 2100
@@
 F 0 "SW8" H 3550 2210 50  0000 C CNN
 F 1 "MINUS" V 3400 2020 50  0000 C CNN
-F 2 "Keyboard:CHERRY_PLATE_100H" H 3400 2100 50  0001 C CNN
+F 2 "Tim's Cherry MX:CHERRY_PLATE_100H" H 3400 2100 50  0001 C CNN
 F 3 "" H 3400 2100 50  0000 C CNN
 	1    3400 2100
@@
 F 0 "SW6" H 2150 2210 50  0000 C CNN
 F 1 "SLASH" V 2000 2020 50  0000 C CNN
-F 2 "Keyboard:CHERRY_PLATE_100H" H 2000 2100 50  0001 C CNN
+F 2 "Tim's Cherry MX:CHERRY_PLATE_100H" H 2000 2100 50  0001 C CNN
 F 3 "" H 2000 2100 50  0000 C CNN
 	1    2000 2100
@@
 F 0 "SW9" H 1450 3410 50  0000 C CNN
 F 1 "7" V 1300 3220 50  0000 C CNN
-F 2 "Keyboard:CHERRY_PLATE_100H" H 1300 3300 50  0001 C CNN
+F 2 "Tim's Cherry MX:CHERRY_PLATE_100H" H 1300 3300 50  0001 C CNN
 F 3 "" H 1300 3300 50  0000 C CNN
 	1    1300 3300
@@
 F 0 "SW11" H 2850 3410 50  0000 C CNN
 F 1 "9" V 2700 3220 50  0000 C CNN
-F 2 "Keyboard:CHERRY_PLATE_100H" H 2700 3300 50  0001 C CNN
+F 2 "Tim's Cherry MX:CHERRY_PLATE_100H" H 2700 3300 50  0001 C CNN
 F 3 "" H 2700 3300 50  0000 C CNN
 	1    2700 3300
@@
 F 0 "SW12" H 3550 3410 50  0000 C CNN
 F 1 "PLUS" V 3400 3220 50  0000 C CNN
-F 2 "Keyboard:CHERRY_PLATE_200V" H 3400 3300 50  0001 C CNN
+F 2 "Tim's Cherry MX:CHERRY_PLATE_200V" H 3400 3300 50  0001 C CNN
 F 3 "" H 3400 3300 50  0000 C CNN
 	1    3400 3300
@@
 F 0 "SW10" H 2150 3410 50  0000 C CNN
 F 1 "8" V 2000 3220 50  0000 C CNN
-F 2 "Keyboard:CHERRY_PLATE_100H" H 2000 3300 50  0001 C CNN
+F 2 "Tim's Cherry MX:CHERRY_PLATE_100H" H 2000 3300 50  0001 C CNN
 F 3 "" H 2000 3300 50  0000 C CNN
 	1    2000 3300
@@
 F 0 "SW13" H 1450 4610 50  0000 C CNN
 F 1 "4" V 1300 4420 50  0000 C CNN
-F 2 "Keyboard:CHERRY_PLATE_100H" H 1300 4500 50  0001 C CNN
+F 2 "Tim's Cherry MX:CHERRY_PLATE_100H" H 1300 4500 50  0001 C CNN
 F 3 "" H 1300 4500 50  0000 C CNN
 	1    1300 4500
@@
 F 0 "SW15" H 2850 4610 50  0000 C CNN
 F 1 "6" V 2700 4420 50  0000 C CNN
-F 2 "Keyboard:CHERRY_PLATE_100H" H 2700 4500 50  0001 C CNN
+F 2 "Tim's Cherry MX:CHERRY_PLATE_100H" H 2700 4500 50  0001 C CNN
 F 3 "" H 2700 4500 50  0000 C CNN
 	1    2700 4500
@@
 F 0 "SW16" H 3550 4610 50  0000 C CNN
 F 1 "ENTER" V 3400 4420 50  0000 C CNN
-F 2 "Keyboard:CHERRY_PLATE_200V" H 3400 4500 50  0001 C CNN
+F 2 "Tim's Cherry MX:CHERRY_PLATE_200V" H 3400 4500 50  0001 C CNN
 F 3 "" H 3400 4500 50  0000 C CNN
 	1    3400 4500
@@
 F 0 "SW14" H 2150 4610 50  0000 C CNN
 F 1 "5" V 2000 4420 50  0000 C CNN
-F 2 "Keyboard:CHERRY_PLATE_100H" H 2000 4500 50  0001 C CNN
+F 2 "Tim's Cherry MX:CHERRY_PLATE_100H" H 2000 4500 50  0001 C CNN
 F 3 "" H 2000 4500 50  0000 C CNN
 	1    2000 4500
@@
 F 0 "SW17" H 1450 5710 50  0000 C CNN
 F 1 "1" V 1300 5520 50  0000 C CNN
-F 2 "Keyboard:CHERRY_PLATE_100H" H 1300 5600 50  0001 C CNN
+F 2 "Tim's Cherry MX:CHERRY_PLATE_100H" H 1300 5600 50  0001 C CNN
 F 3 "" H 1300 5600 50  0000 C CNN
 	1    1300 5600
@@
 F 0 "SW19" H 2850 5710 50  0000 C CNN
 F 1 "3" V 2700 5520 50  0000 C CNN
-F 2 "Keyboard:CHERRY_PLATE_100H" H 2700 5600 50  0001 C CNN
+F 2 "Tim's Cherry MX:CHERRY_PLATE_100H" H 2700 5600 50  0001 C CNN
 F 3 "" H 2700 5600 50  0000 C CNN
 	1    2700 5600
@@
 F 0 "SW20" H 3550 5710 50  0000 C CNN
 F 1 "0" V 3400 5520 50  0000 C CNN
-F 2 "Keyboard:CHERRY_PLATE_200H" H 3400 5600 50  0001 C CNN
+F 2 "Tim's Cherry MX:CHERRY_PLATE_200H" H 3400 5600 50  0001 C CNN
 F 3 "" H 3400 5600 50  0000 C CNN
 	1    3400 5600
@@
 F 0 "SW18" H 2150 5710 50  0000 C CNN
 F 1 "2" V 2000 5520 50  0000 C CNN
-F 2 "Keyboard:CHERRY_PLATE_100H" H 2000 5600 50  0001 C CNN
+F 2 "Tim's Cherry MX:CHERRY_PLATE_100H" H 2000 5600 50  0001 C CNN
 F 3 "" H 2000 5600 50  0000 C CNN
 	1    2000 5600
@@
 F 0 "SW21" H 4250 5710 50  0000 C CNN
 F 1 "PERIOD" V 4100 5520 50  0000 C CNN
-F 2 "Keyboard:CHERRY_PLATE_100H" H 4100 5600 50  0001 C CNN
+F 2 "Tim's Cherry MX:CHERRY_PLATE_100H" H 4100 5600 50  0001 C CNN
 F 3 "" H 4100 5600 50  0000 C CNN
 	1    4100 5600
